File: Modules/CaptainsLog/CaptainsLog.kicad_sch (KiCad schematic)
At the start: 52 parts, among them J1 Conn_01x12, J2 Micro_SD_Card, J3 Micro_SD_Card, U2 FSSD06

Commit message: Reset Push
Git deleted work. Restarting layout with schematic modifications. Renamed board
Parts:
- removed D3, D7: SP3011, watchstander:SP3011-06UTG, symbol watchstander:SP3011
- removed J2, J3: Micro_SD_Card, watchstander:GCT_MEM2052, symbol watchstander:Micro_SD_Card
- removed R10, R11, R28, R29, R30, R7: 0, Resistor_SMD:R_0201_0603Metric, symbol Device:R
- removed TP19, TP20: TestPoint, TestPoint:TestPoint_THTPad_2.0x2.0mm_Drill1.0mm, symbol Connector:TestPoint
- removed U2: FSSD06, watchstander:FSSD06, symbol watchstander:FSSD06BQX
- added D1, D2: SP3011, CaptainsLog:SP3011-06UTG, symbol CaptainsLog:SP3011
- added J4, J5: Micro_SD_Card, CaptainsLog:GCT_MEM2052, symbol CaptainsLog:Micro_SD_Card
- added U1: FSSD06, CaptainsLog:FSSD06, symbol CaptainsLog:FSSD06BQX
- H1, H2, H3, H4: footprint MountingHole:MountingHole_2.5mm_Pad -> MountingHole:MountingHole_2.2mm_M2
- R12, R6: footprint Resistor_SMD:R_0603_1608Metric -> Resistor_SMD:R_0201_0603Metric
Connections:
- net MUX_CLK is gone; now on net SD_CLK_IN: TP4.1
- net MUX_D1 is gone; now on net SD_CMD_IN: TP3.1
- net +V_SD1: now also J5.4 (VDD), U1.22 (SD1_VDDC)
- net +V_SD2: now also J4.4 (VDD), U1.15 (SD2_VDDC)
- net GND: now also D1.10, D1.5, D2.10, D2.5, J4.6 (VSS), J4.SH (SHIELD), J5.6 (VSS), J5.SH (SHIELD), U1.7 (GND)
- net MUX_OE: now also U1.2 (OE)
- net MUX_SEL: now also U1.11 (SD_Sel)
- net SD1_CLK: now also D1.11 (Conn4), D1.4 (Conn4), J5.5 (CLK), U1.21 (SD1_CLK)
- net SD1_CMD: now also D1.12 (Conn3), D1.3 (Conn3), J5.3 (CMD), U1.23 (SD1_CMD)
- net SD1_DAT0: now also D1.6 (Conn5), D1.9 (Conn5), J5.7 (DAT0), U1.20 (SD1_DAT0)
- net SD1_DAT1: now also D1.7 (Conn6), D1.8 (Conn6), J5.8 (DAT1), U1.19 (SD1_DAT1)
- net SD1_DAT2: now also D1.1 (Conn1), D1.14 (Conn1), J5.1 (DAT2), U1.1 (SD1_DAT2)
- net SD1_DAT3: now also D1.13 (Conn2), D1.2 (Conn2), J5.2 (DAT3/CD), U1.24 (SD1_DAT3)
- net SD1_Det: now also J5.9 (DET)
- net SD2_CLK: now also D2.11 (Conn4), D2.4 (Conn4), J4.5 (CLK), U1.14 (SD2_CLK)
- net SD2_CMD: now also D2.12 (Conn3), D2.3 (Conn3), J4.3 (CMD), U1.16 (SD2_CMD)
- net SD2_DAT0: now also D2.6 (Conn5), D2.9 (Conn5), J4.7 (DAT0), U1.13 (SD2_DAT0)
- net SD2_DAT1: now also D2.7 (Conn6), D2.8 (Conn6), J4.8 (DAT1), U1.12 (SD2_DAT1)
- net SD2_DAT2: now also D2.1 (Conn1), D2.14 (Conn1), J4.1 (DAT2), U1.18 (SD2_DAT2)
- net SD2_DAT3: now also D2.13 (Conn2), D2.2 (Conn2), J4.2 (DAT3/CD), U1.17 (SD2_DAT3)
- net SD2_Det: now also J4.9 (DET)
- net SD_CLK_IN: now also U1.8 (CLK)
- net SD_CMD_IN: now also U1.5 (CMD)
- net SD_DAT0_IN: now also U1.9 (DAT0)
- net SD_DAT1_IN: now also U1.10 (DAT1)
- net SD_DAT2_IN: now also U1.3 (DAT2)
- net SD_DAT3_IN: now also U1.4 (DAT3)
- net Vin: now also U1.6 (VDDH)
Other:
- note added: "Captain's Log"
- note added: "PWR Indicators"
- note removed: "PWR Indicator"
- note removed: "SD PWR Indicators"
- note removed: "Watchstander"
- title: Watchstander uSD Breakout Board -> Captain's Log uSD Board
- moved on the sheet: D5, H1, H2, H3, H4, R1, R12, R2, R25, R3, R4, R5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
